File: Hardware/SolarMonitorMainBoard/SolarMonitorMainBoard.brd (EAGLE design)
At the start: 100 x 80 mm, 28 parts, among them U1 INA219AIDR, U2 INA219AIDR, U3 INA219AIDR, U4 INA219AIDR, U5 INA219AIDR, U6 TSR_1-2450, X1 MKDS_5/3-7,62, X2 MKDS_5/3-7,62, X3 MKDS_5/3-7,62, X4 MKDS_5/3-7,62

Commit message: Work in progress on the main board ...
Parts:
- removed R8: (no value), resistor-shunt:SMV
- added K1: RT314F12, relay:RT1-BI
- R1, R2, R3, R4, R5: value (none) -> 5m; device adafruit:R2512 -> resistor-shunt:SMV
- moved U4 2.84 mm to (74.9, 27.9)
- moved C5 2.84 mm to (85.1, 26.0)
- moved J1 2.84 mm to (52.1, 33.0)
- moved U3 2.84 mm to (58.4, 27.9)
- moved C3 2.84 mm to (53.3, 26.0)
- moved R6 2.84 mm to (48.3, 27.9)
- moved R7 2.84 mm to (48.9, 24.1)
- moved U2 2.84 mm to (41.9, 27.9)
- moved U5 2.84 mm to (90.2, 27.9)
- moved C2 2.84 mm to (36.8, 26.0)
- moved C4 2.84 mm to (69.8, 26.0)
- moved R1 2.62 mm to (26.0, 18.4), turned to 0 degrees
- moved U1 2.54 mm to (25.4, 27.9)
- moved C1 2.54 mm to (20.3, 26.0)
- moved R4 2.01 mm to (74.3, 18.4), turned to 0 degrees
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Connections:
- new net N$11: R2.U1, U2.8
- new net N$12: R2.U2, U2.7
- new net N$13: R1.U1, U1.8
- new net N$14: R1.U2, U1.7
- new net N$15: R3.U1, U3.8
- new net N$16: R3.U2, U3.7
- new net N$17: R4.U1, U4.8
- new net N$18: R4.U2, U4.7
- new net N$19: R5.U1, U5.8
- new net N$20: R5.U2, U5.7
- net 1VIN+: now also R1.I1; no longer R1.1, U1.8
- net 1VIN-: now also R1.I2; no longer R1.2, U1.7
- net N$1: now also R2.I2; no longer R2.2, U2.7
- net N$10: now also R5.I2; no longer R5.2, U5.7
- net N$4: now also R2.I1; no longer R2.1, U2.8
- net N$5: now also R3.I1; no longer R3.1, U3.8
- net N$6: now also R3.I2; no longer R3.2, U3.7
- net N$7: now also R4.I2; no longer R4.2, U4.7
- net N$8: now also R4.I1; no longer R4.1, U4.8
- net N$9: now also R5.I1; no longer R5.1, U5.8

Commit message: Work in progress on the main board ...
Parts:
- removed MS2: FONA, BtParts:FONA
- removed R7: (no value), SparkFun-Resistors:0805
- added C6: (no value), SparkFun-Capacitors:0805
- added D2, D3: (no value), diode:SMB
- added J2: (no value), SparkFun-Connectors:2X10
- added K2: RT314F12, relay:RT1-BI
- added R10, R11: (no value), SparkFun-Resistors:0805
- added U10: TSR_1-2450, _traco_tsr-1:TSR-1
- added U7: MCP23008-E/SS, Microchip_By_element14_Batch_1:SOP65P780X200-20N
- added U8: ULN2803ADW, Texas Instruments_By_element14_Batch_1:SOIC127P1030X265-18N
- MS1: value FEATHERWING -> FEATHERWING_NODIM; device adafruit:FEATHERWING -> adafruit:FEATHERWING_DIM
- R6: value (none) -> 5m; device SparkFun-Resistors:0805 -> resistor-shunt:SMV
- U6: value TSR_1-2450 -> INA219AIDR; device _traco_tsr-1:TSR-1 -> Texas Instruments_By_element14_Batch_1:SOIC127P600X175-8N
- moved U6 80.7 mm to (89.5, 21.6), turned to 180 degrees
- moved U$1 35.6 mm to (52.1, 61.0)
- moved R6 33.3 mm to (80.6, 20.3), turned to 270 degrees
- moved J1 31.5 mm to (66.7, 61.0)
- moved U5 27.9 mm to (62.2, 27.9)
- moved D1 27.7 mm to (59.1, 59.1)
- moved C5 24.3 mm to (61.0, 23.5), turned to 180 degrees
- moved R5 20.4 mm to (69.8, 20.3), turned to 270 degrees
- moved U4 19.7 mm to (55.2, 29.2)
- moved U3 17.8 mm to (40.6, 29.2)
- moved U1 17.8 mm to (7.62, 29.2)
- moved U2 17.8 mm to (24.1, 29.2)
- moved R4 17.1 mm to (57.1, 18.4)
- moved R3 16.5 mm to (41.9, 18.4)
- moved R1 16.5 mm to (9.53, 18.4)
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Connections:
- new net FONA_RX: J2.8, MS1.15
- new net FONA_TX: J2.6, MS1.14
- new net LIN1: D2.A, K1.12B, R5.I2
- new net LIN2: D3.A, K1.14B, R6.I2
- new net LOUT: K2.14A, X4.3
- new net N$21: R6.I1, X4.1
- new net N$22: K1.11A, K2.11B
- new net N$23: R6.U1, U6.8
- new net N$24: R6.U2, U6.7
- new net N$25: U7.16, U8.4
- new net N$26: U7.15, U8.5
- new net N$27: U7.14, U8.6
- new net N$28: U7.13, U8.7
- new net N$29: U7.12, U8.8
- new net N$30: K2.A1, U8.11
- new net N$31: K2.A2, U8.12
- new net N$32: K1.A1, U8.13
- new net N$33: K1.A2, U8.14
- net 1VIN+: now also X1.2; no longer X2.1
- net 1VIN-: now also X1.1; no longer X1.3
- net 5V: now also J2.2, U10.3; no longer MS2.99, U6.3
- net FONA_BAT: now also J2.4; no longer MS2.1
- net FONA_RST: now also J2.10; no longer MS2.5
- net GND: now also C6.1, J2.1, K1.A3, K2.A3, U10.2, U6.6, U7.3, U7.4, U7.5, U7.9, U8.9; no longer MS2.2, X1.2
- net N$1: now also X1.3; no longer X2.2
- net N$10: now also U7.17, U8.3; no longer R5.I2, X4.2
- net N$2: now also U7.19, U8.1; no longer MS1.15, MS2.10
- net N$3: now also U7.18, U8.2; no longer MS1.14, MS2.9
- net N$4: now also X2.1; no longer X2.3
- net N$5: now also X2.3; no longer X3.2
- net N$6: now also X2.2; no longer X3.1
- net N$7: now also X3.1; no longer X3.3
- net N$8: now also X3.2; no longer X4.1
- net N$9: now also X3.3; no longer X4.3
- net SCL: now also R10.1, U6.4, U7.1; no longer R6.1
- net SDA: now also R11.2, U6.1, U6.3, U7.2; no longer R7.2
- net VCC: now also C6.2, J2.3, R10.2, R11.1, U6.5, U7.20, U7.6; no longer MS2.12, R6.2, R7.1
- net VI: now also D2.C, D3.C, U10.1, U8.10; no longer U6.1, X1.1
Routing:
- net VCC: track 0.00 -> 85.8 mm
- net VI: track 0.00 -> 53.9 mm
- net LIN2: track 0.00 -> 32.2 mm, vias 0 -> 1
- net N$32: track 0.00 -> 30.3 mm
- net LIN1: track 0.00 -> 28.4 mm
- net LOUT: track 0.00 -> 23.1 mm
- net N$30: track 0.00 -> 19.1 mm
- net GND: track 0.00 -> 18.2 mm
- net N$20: track 0.00 -> 17.6 mm
- net N$33: track 0.00 -> 17.0 mm
- net N$31: track 0.00 -> 16.8 mm
- net SDA: track 0.00 -> 12.9 mm
- net N$13: track 0.00 -> 12.8 mm
- net N$11: track 0.00 -> 12.8 mm
- net N$17: track 0.00 -> 12.8 mm
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- added copper zone on layer 1, net GND
Other:
- board size 100 x 80 mm -> 100 x 78.7 mm

Commit message: Work in progress on the main board ...
Parts:
- moved U6 98.0 mm to (5.71, 72.4)
- moved R6 80.3 mm to (18.4, 71.1), turned to 180 degrees
- moved C6 76.5 mm to (27.9, 74.9), turned to 270 degrees
- moved J1 33.6 mm to (33.7, 67.3)
- moved D1 29.5 mm to (32.4, 71.8)
- moved C5 27.3 mm to (87.0, 15.2)
- moved R5 24.3 mm to (94.1, 20.3), turned to 90 degrees
- moved U5 24.1 mm to (84.7, 19.3), turned to 0 degrees
- moved U1 8.27 mm to (15.9, 29.7)
- moved U2 7.38 mm to (31.5, 29.7)
- moved U4 7.13 mm to (62.4, 29.7)
- moved C1 6.73 mm to (12.4, 24.8)
- moved U3 6.50 mm to (47.1, 29.7)
- moved R1 6.36 mm to (15.9, 18.7)
- moved X1 6.10 mm to (20.1, 8.26)
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Connections:
- removed net LOUT: K2.14A, X4.3
- removed net N$21: R6.I1, X4.1
- removed net N$9: R5.I1, X3.3
- new net LOUT+: K2.14A, R5.I1
- new net LOUT-: R5.I2, X4.3
- net LIN1: now also X3.3; no longer R5.I2
- net LIN2: now also X4.1; no longer R6.I2
Routing:
- net SCL: track 2.90 -> 115.2 mm, vias 0 -> 5
- net SDA: track 12.9 -> 103.9 mm, vias 0 -> 2
- net VCC: track 85.8 -> 134.6 mm, vias 0 -> 2
- net LOUT: track 23.1 -> 0.00 mm
- net LIN1: track 28.4 -> 47.3 mm
- net LIN2: track 32.2 -> 48.3 mm
- net N$20: track 17.6 -> 2.91 mm
- net N$23: track 10.6 -> 0.00 mm
- net GND: track 18.2 -> 26.4 mm, vias 0 -> 5
- net LOUT-: track 0.00 -> 7.38 mm
- net N$21: track 7.31 -> 0.00 mm
- net N$9: track 7.06 -> 0.00 mm
- net LOUT+: track 0.00 -> 5.77 mm
- net VI: track 53.9 -> 59.0 mm
- net N$19: track 6.23 -> 11.1 mm
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- added copper zone on layer 16, net GND

Commit message: Work in progress on the main board ...
Parts:
- added C7: (no value), SparkFun-Capacitors:0805
- added R7: (no value), SparkFun-Resistors:R2512
- added R8: (no value), SparkFun-Resistors:0805
- added X6: MKDSN1,5/8-5,08, con-phoenix-508:MKDSN1,5/8-5,08
- D2, D3: value (none) -> MBRA140; device diode:SMB -> SparkFun-DiscreteSemi:SMA-DIODE
- R6: value 5m -> (none); device resistor-shunt:SMV -> SparkFun-Resistors:0805
- U7: value MCP23008-E/SS -> ATMEGA328P_TQFP; device Microchip_By_element14_Batch_1:SOP65P780X200-20N -> SparkFun-DigitalIC:TQFP32-08
- moved R6 79.4 mm to (97.8, 69.8), turned to 0 degrees
- moved U6 64.7 mm to (66.7, 50.8)
- moved R11 63.2 mm to (5.08, 32.5)
- moved R10 63.2 mm to (8.00, 29.7), turned to 180 degrees
- moved C6 40.7 mm to (61.8, 52.5), turned to 90 degrees
- moved D1 31.4 mm to (54.0, 48.9), turned to 270 degrees
- moved J1 30.6 mm to (54.0, 44.5), turned to 270 degrees
- moved J2 5.08 mm to (21.6, 62.2), turned to 180 degrees
- moved U$1 4.55 mm to (56.0, 58.7)
- moved U10 4.17 mm to (63.5, 57.9)
- moved U7 1.42 mm to (70.1, 70.0), turned to 90 degrees
- moved U8 1.27 mm to (85.1, 68.6)
- turned D2 to 90 degrees
- turned D3 to 90 degrees
Connections:
- new net DISP1_CE: J2.8, MS1.9
- new net DISP1_RST: J2.6, MS1.8
- new net DISP2_CE: J2.4, MS1.7
- new net DISP2_RST: J2.2, MS1.6
- new net DISP_DC: J2.10, MS1.10
- new net N$21: U7.11, U8.6
- new net N$34: J2.13
- new net N$35: J2.11
- new net N$36: J2.9
- new net N$37: D1.C, J1.1
- new net N$9: D2.C, D3.C, R7.2, U6.8
- new net T_A_B: U7.1, X6.3
- new net T_ON_OFF: U7.32, X6.2
- net 5V: now also J2.5; no longer J2.2
- net FONA_BAT: now also J2.7; no longer J1.1, J2.4
- net FONA_RST: no longer J2.10
- net FONA_RX: now also J2.20; no longer J2.8
- net FONA_TX: now also J2.18; no longer J2.6
- net GND: now also C7.1, X4.2, X6.1; no longer U7.4, U7.9
- net LOUT+: now also R6.2
- net MISO: now also J2.16
- net MOSI: now also J2.14
- net N$10: now also U7.10, U8.7; no longer U7.17, U8.3
- net N$2: now also R6.1, R8.2, U7.2; no longer U7.19, U8.1
- net N$23: now also U7.12, U8.5; no longer R6.U1, U6.8
- net N$24: now also U7.13, U8.4; no longer R6.U2, U6.7
- net N$25: now also U7.14, U8.3; no longer U7.16, U8.4
- net N$26: now also R8.1; no longer U7.15, U8.5
- net N$27: now also J2.19; no longer U7.14, U8.6
- net N$28: now also J2.17; no longer U7.13, U8.7
- net N$29: now also J2.15; no longer U7.12, U8.8
- net N$3: now also U7.9, U8.8; no longer U7.18, U8.2
- net SCK: now also J2.12
- net SCL: now also U7.28; no longer U7.1
- net SDA: now also U7.27; no longer U7.2
- net VBAT: no longer D1.C
- net VCC: now also C7.2, U7.18, U7.4; no longer U7.20
- net VI: now also R7.1, U6.7; no longer D2.C, D3.C
Routing:
- net VCC: track 134.6 -> 244.2 mm
- net 5V: track 0.00 -> 88.0 mm
- net N$9: track 0.00 -> 18.5 mm
- net SDA: track 103.9 -> 115.8 mm, vias 2 -> 4
- net SCL: track 115.2 -> 124.5 mm
- net N$2: track 6.85 -> 0.00 mm
- net N$21: track 0.00 -> 6.50 mm
- net N$29: track 6.32 -> 0.00 mm
- net N$23: track 0.00 -> 6.29 mm
- net N$24: track 0.00 -> 6.10 mm
- net N$28: track 6.07 -> 0.00 mm
- net N$26: track 5.83 -> 0.00 mm
- net N$27: track 5.82 -> 0.00 mm
- net N$30: track 19.1 -> 13.4 mm
- net SCK: track 0.00 -> 5.08 mm
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
Commit message: Update schematic
Parts:
- added K3: RT314F12, relay:RT1-BI
- added R12, R13, R14, R9: (no value), SparkFun-Resistors:0805
- added X5: MKDS_5/3-7,62, con-phoenix-mkds_5:MKDS_5/3-762
- moved K1 84.9 mm to (12.7, -10.2), turned to 0 degrees
- moved K2 14.0 mm to (78.7, 43.2)
Connections:
- new net LIN1SENSE: K1.14A, K1.14B, R9.2
- new net LIN2SENSE: K2.12A, K2.12B, R13.2
- new net N$38: R12.2, R9.1, U7.24
- new net N$39: R12.1
- new net N$40: R13.1, R14.2, U7.25
- new net N$41: R14.1
- new net N$42: K1.A1, U8.15
- new net N$43: K1.A2, U8.16
- net GND: now also K3.A3; no longer K1.A3
- net LIN1: now also K1.11A, K1.11B, X5.1; no longer K1.12B, X3.3
- net LIN2: now also K2.11A, K2.11B, X5.2; no longer K1.14B, X4.1
- net LOUT+: now also K3.14A, K3.14B; no longer K2.14A
- net LOUT-: now also X5.3; no longer X4.3
- net N$2: now also U7.23; no longer U7.2
- net N$22: now also K1.12A, K1.12B, K2.14A, K2.14B, K3.11A, K3.11B; no longer K1.11A, K2.11B
- net N$30: now also K3.A1; no longer K2.A1
- net N$31: now also K3.A2; no longer K2.A2
- net N$32: now also K2.A1; no longer K1.A1
- net N$33: now also K2.A2; no longer K1.A2
Routing:
- net LIN2: track 48.3 -> 7.88 mm
- net LIN1: track 47.3 -> 32.9 mm
- net LOUT-: track 7.38 -> 0.00 mm
- net N$22: track 6.41 -> 0.00 mm

Commit message: Lets hope
Parts:
- removed X4: MKDS_5/3-7,62, con-phoenix-mkds_5:MKDS_5/3-762
- added J3: (no value), SparkFun-Connectors:2X4
- moved X5 124.2 mm to (74.4, 70.7), turned to 180 degrees
- moved K1 108.9 mm to (93.2, 63.1), turned to 90 degrees
- moved R14 98.0 mm to (83.8, 24.1)
- moved R12 97.8 mm to (85.1, 26.7)
- moved R8 94.6 mm to (8.89, 38.1)
- moved R6 92.4 mm to (10.2, 40.6)
- moved R9 92.2 mm to (80.0, 26.7)
- moved R13 91.2 mm to (74.9, 27.9)
- moved C5 64.3 mm to (47.6, 66.0)
- moved U5 64.3 mm to (45.3, 70.1), turned to 90 degrees
- moved R5 63.1 mm to (54.7, 69.6), turned to 270 degrees
- moved J1 56.1 mm to (1.65, 64.6)
- moved D1 55.6 mm to (1.65, 67.8)
- moved U$1 51.1 mm to (85.2, 16.8), turned to 0 degrees
- moved U7 50.0 mm to (93.0, 25.5), turned to 180 degrees
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Connections:
- net GND: now also X3.3; no longer X4.2
Routing:
- net VCC: track 244.2 -> 34.7 mm, vias 2 -> 0
- net SCL: track 124.5 -> 7.02 mm, vias 5 -> 0
- net SDA: track 115.8 -> 4.84 mm, vias 4 -> 0
- net 5V: track 88.0 -> 0.00 mm
- net LIN2: track 7.88 -> 67.7 mm, vias 1 -> 0
- net VI: track 60.5 -> 7.48 mm
- net N$22: track 0.00 -> 39.0 mm
- net N$32: track 31.5 -> 0.00 mm
- net LIN1: track 32.9 -> 61.1 mm, vias 0 -> 1
- net N$33: track 18.3 -> 0.00 mm
- net N$31: track 15.5 -> 0.00 mm
- net LOUT-: track 0.00 -> 15.2 mm
- net N$30: track 13.4 -> 0.00 mm
- net N$20: track 2.91 -> 14.6 mm
- net LOUT+: track 5.77 -> 14.7 mm
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
Commit message: Before autoroute try
Parts:
- added C8: (no value), SparkFun-Capacitors:0805
- MS1: device adafruit:FEATHERWING_DIM -> BtParts:FEATHERWING_DIM
- moved R8 69.3 mm to (77.5, 27.9)
- moved C7 54.6 mm to (83.8, 27.6)
- moved R13 13.5 mm to (85.1, 19.1), turned to 180 degrees
- moved C5 8.89 mm to (47.6, 74.9), turned to 0 degrees
- moved R12 5.39 mm to (81.3, 22.9), turned to 90 degrees
- moved R9 4.58 mm to (77.5, 22.9), turned to 180 degrees
- moved R14 3.19 mm to (85.1, 21.2)
- moved J3 1.45 mm to (77.1, 16.4), turned to 180 degrees
- moved U7 1.27 mm to (91.7, 25.5)
- moved U5 1.14 mm to (46.4, 69.6)
Connections:
- removed net N$30: K3.A1, U8.11
- removed net N$31: K3.A2, U8.12
- removed net N$39: R12.1
- removed net N$41: R14.1
- new net N$45: K1.A1, U8.11
- new net N$47: K3.A1, U8.16
- net GND: now also C8.1, K1.A3, R12.1, R14.1
- net N$42: now also K3.A2; no longer K1.A1
- net N$43: now also U8.12; no longer U8.16
- net VCC: now also C8.2
Routing:
- net VI: track 7.48 -> 64.3 mm, vias 0 -> 1
- net N$42: track 0.00 -> 36.2 mm
- net N$47: track 0.00 -> 28.3 mm
- net N$33: track 0.00 -> 26.9 mm
- net N$32: track 0.00 -> 21.0 mm
- net VCC: track 34.7 -> 55.1 mm
- net N$43: track 0.00 -> 10.4 mm
- net GND: track 26.4 -> 18.4 mm
- net N$45: track 0.00 -> 6.57 mm
- net N$25: track 0.00 -> 5.82 mm
- net N$24: track 0.00 -> 5.71 mm
- net N$3: track 0.00 -> 5.53 mm
- net N$23: track 0.00 -> 5.50 mm
- net N$10: track 0.00 -> 5.47 mm
- net N$21: track 0.00 -> 5.33 mm
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
Commit message: Schematic done. Lets route ...
Parts:
- removed J1: (no value), SparkFun-Connectors:1X02
- added D21, D22, D23: 3.3V, SparkFun-DiscreteSemi:SOD-323
- added R21: (no value), SparkFun-Resistors:0805
- C7, C8: value (none) -> 0.1uF
- J2: device SparkFun-Connectors:2X10 -> SparkFun-Connectors:2X8
- R6: value (none) -> 10k
- moved R6 84.1 mm to (91.4, 19.1)
- moved U10 28.7 mm to (6.86, 63.4)
- moved D1 22.9 mm to (24.5, 67.8)
- moved J2 16.9 mm to (33.0, 64.5)
- moved R10 0.65 mm to (6.22, 30.2)
- renumbered R13 to R23, R9 to R22
Connections:
- net D6 renamed SD_CARD_DETECT
- removed net N$26: R8.1
- removed net N$27: J2.19
- removed net N$28: J2.17
- removed net N$29: J2.15
- removed net N$34: J2.13
- removed net N$35: J2.11
- removed net N$36: J2.9
- removed net N$37: D1.C, J1.1
- new net FONA_KEY: J2.9, MS1.24
- new net FONA_PS: J2.11, MS1.5
- new net MASTER_EXT_IO: MS1.25, X6.8
- new net N$30: U7.19, U8.1
- new net N$31: U7.22, U8.2
- new net OUT_12V_1: U8.18, X6.4
- new net OUT_12V_2: U8.17, X6.5
- new net SLAVE_EXT_IO: U7.26, X6.7
- new net SLAVE_GND: J3.6
- new net SLAVE_MISO: J3.1, U7.16
- new net SLAVE_MOSI: J3.4, U7.15
- new net SLAVE_NOTIFY: MS1.19, U7.2
- new net SLAVE_RESET: J3.5, MS1.23, R6.1, U7.29
- new net SLAVE_RX: J3.7, U7.30
- new net SLAVE_SCK: J3.3, U7.17
- new net SLAVE_TX: J3.8, U7.31
- new net SLAVE_VCC: J3.2
- net FONA_RX: now also J2.15; no longer J2.20
- net FONA_TX: now also J2.13; no longer J2.18
- net GND: now also D21.A, D22.A, D23.A, R8.1, U7.21
- net LOUT+: now also R21.2; no longer R6.2
- net LOUT-: now also X6.6
- net N$2: now also D21.C, R21.1; no longer R6.1
- net N$38: now also D22.C
- net N$40: now also D23.C
- net VBAT: now also D1.C; no longer J1.2
- net VCC: now also R6.2
Routing:
- net VCC: track 55.1 -> 134.5 mm
- net SCL: track 7.02 -> 66.2 mm, vias 0 -> 3
- net FONA_TX: track 8.18 -> 0.00 mm
- net FONA_RX: track 8.18 -> 0.00 mm
- net N$25: track 5.82 -> 0.00 mm
- net N$24: track 5.71 -> 0.00 mm
- net N$3: track 5.53 -> 0.00 mm
- net N$23: track 5.50 -> 0.00 mm
- net N$10: track 5.47 -> 0.00 mm
- net N$21: track 5.33 -> 0.00 mm
- net VI: track 64.3 -> 67.2 mm, vias 1 -> 0
- net DISP2_RST: track 8.18 -> 6.10 mm
- net DISP2_CE: track 8.18 -> 6.10 mm
- net DISP1_RST: track 8.18 -> 6.10 mm
- net SCK: track 8.18 -> 6.10 mm
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