File: Hardware/SolarMonitorMainBoard/SolarMonitorMainBoard.brd (EAGLE design)
At the start: 100 x 78.7 mm, 51 parts, among them J2 ToTopPrint, J3 ISP, K1 RT314F12, K2 RT314F12, K3 RT314F12, U1 INA219AIDR, U10 TSR_1-2450, U2 INA219AIDR, U3 INA219AIDR, U4 INA219AIDR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

Commit message: Work in progress.
Other:
- board text added: "Rx"
- board text added: "bittailor - SolarMonitor Main Board - rev A"
- board text removed: "RX"
- board text removed: "rev A"
Changed lines of the file:
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@@
 <text x="81.28" y="64.77" size="1.016" layer="21" rot="SR0">L1in</text>
 <text x="14.732" y="48.133" size="1.6764" layer="21" font="vector">BT SolarMonitor</text>
-<text x="90.17" y="2.54" size="1.016" layer="22" rot="MR0">rev A</text>
+<text x="90.17" y="2.54" size="1.016" layer="22" rot="MR0">bittailor - SolarMonitor Main Board - rev A</text>
 <wire x1="71.755" y1="64.135" x2="84.455" y2="64.135" width="0.127" layer="21"/>
 <wire x1="84.455" y1="64.135" x2="84.455" y2="68.58" width="0.127" layer="21"/>
@@
 <text x="1.524" y="69.215" size="1.016" layer="21" rot="SR0">IO2</text>
 <text x="79.121" y="14.351" size="1.016" layer="21">ISP</text>
-<text x="78.74" y="2.413" size="1.016" layer="21">RX</text>
+<text x="78.74" y="2.413" size="1.016" layer="21">Rx</text>
 <text x="81.407" y="2.413" size="1.016" layer="21">Tx</text>
 <text x="70.231" y="13.716" size="1.016" layer="21">GND</text>

Commit message: Fix ground instead of +12V error in schematic routing on board not done yet.
Connections:
- net GND: no longer K1.A3, K2.A3, K3.A3
- net VI: now also K1.A3, K2.A3, K3.A3
Changed lines of the file:
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@@
 <contactref element="J2" pad="1"/>
 <contactref element="U8" pad="9"/>
-<contactref element="K3" pad="A3"/>
-<contactref element="K2" pad="A3"/>
 <contactref element="C6" pad="1"/>
 <wire x1="27.189" y1="24.638" x2="28.956" y2="25.019" width="0.254" layer="1"/>
@@
 <wire x1="39.889" y1="44.069" x2="40.005" y2="46.4312" width="0.254" layer="1"/>
 <contactref element="X3" pad="3"/>
-<contactref element="K1" pad="A3"/>
 <contactref element="R22" pad="1"/>
 <contactref element="R23" pad="1"/>
@@
 <wire x1="49.53" y1="37.846" x2="37.592" y2="37.846" width="0.6096" layer="1"/>
 <wire x1="37.592" y1="37.846" x2="34.417" y2="40.64" width="0.6096" layer="1"/>
+<contactref element="K3" pad="A3"/>
+<contactref element="K2" pad="A3"/>
+<contactref element="K1" pad="A3"/>
+<wire x1="97.917" y1="52.959" x2="93.218" y2="50.519" width="0" layer="19" extent="1-1"/>
+<wire x1="64.77" y1="38.2" x2="70.358" y2="45.974" width="0" layer="19" extent="1-1"/>
+<wire x1="78.359" y1="33.12" x2="77.47" y2="45.974" width="0" layer="19" extent="1-1"/>
 </signal>
 <signal name="5V">
