File: Hardware/SolarMonitorMainBoard/SolarMonitorMainBoard.sch (EAGLE design)
At the start: 28 parts, among them U1 INA219AIDR, U2 INA219AIDR, U3 INA219AIDR, U4 INA219AIDR, U5 INA219AIDR, U6 TSR_1-2450, X1 MKDS_5/3-7,62, X2 MKDS_5/3-7,62, X3 MKDS_5/3-7,62, X4 MKDS_5/3-7,62

Commit message: Work in progress on the main board ...
Parts:
- removed R8: (no value), resistor-shunt:SMV
- added K1: RT314F12, relay:RT314F12
- R1, R2, R3, R4, R5: value (none) -> 5m; device adafruit:R-US_R2512 -> resistor-shunt:SMV
Connections:
- new net N$11: R2.SA, U2.VIN+
- new net N$12: R2.SB, U2.VIN-
- new net N$13: R1.SA, U1.VIN+
- new net N$14: R1.SB, U1.VIN-
- new net N$15: R3.SA, U3.VIN+
- new net N$16: R3.SB, U3.VIN-
- new net N$17: R4.SA, U4.VIN+
- new net N$18: R4.SB, U4.VIN-
- new net N$19: R5.SA, U5.VIN+
- new net N$20: R5.SB, U5.VIN-
- net 1VIN+: now also R1.A; no longer R1.1, U1.VIN+
- net 1VIN-: now also R1.B; no longer R1.2, U1.VIN-
- net N$1: now also R2.B; no longer R2.2, U2.VIN-
- net N$10: now also R5.B; no longer R5.2, U5.VIN-
- net N$4: now also R2.A; no longer R2.1, U2.VIN+
- net N$5: now also R3.A; no longer R3.1, U3.VIN+
- net N$6: now also R3.B; no longer R3.2, U3.VIN-
- net N$7: now also R4.B; no longer R4.2, U4.VIN-
- net N$8: now also R4.A; no longer R4.1, U4.VIN+
- net N$9: now also R5.A; no longer R5.1, U5.VIN+

Commit message: Work in progress on the main board ...
Parts:
- removed MS2: FONA, BtParts:FONA
- removed R7: (no value), SparkFun-Resistors:RESISTOR0805-RES
- added C6: (no value), SparkFun-Capacitors:CAP0805
- added D2, D3: (no value), diode:SCHOTTKY-DIODESMD
- added J2: (no value), SparkFun-Connectors:M10X2
- added K2: RT314F12, relay:RT314F12
- added R10, R11: (no value), SparkFun-Resistors:RESISTOR0805-RES
- added U10: TSR_1-2450, _traco_tsr-1:TSR_1-2450
- added U7: MCP23008-E/SS, Microchip_By_element14_Batch_1:MCP23008-E/SS
- added U8: ULN2803ADW, Texas Instruments_By_element14_Batch_1:ULN2803ADW
- MS1: value FEATHERWING -> FEATHERWING_NODIM; device adafruit:FEATHERWING -> adafruit:FEATHERWING_NODIM
- R6: value (none) -> 5m; device SparkFun-Resistors:RESISTOR0805-RES -> resistor-shunt:SMV
- U6: value TSR_1-2450 -> INA219AIDR; device _traco_tsr-1:TSR_1-2450 -> Texas Instruments_By_element14_Batch_1:INA219AIDR
Connections:
- new net FONA_RX: J2.8, MS1.GPIOTX
- new net FONA_TX: J2.6, MS1.GPIORX
- new net LIN1: D2.A, K12.OB, R5.B
- new net LIN2: D3.A, K12.SB, R6.B
- new net LOUT: K22.SA, X4-3.KL
- new net N$21: R6.A, X4-1.KL
- new net N$22: K12.PA, K22.PB
- new net N$23: R6.SA, U6.VIN+
- new net N$24: R6.SB, U6.VIN-
- new net N$25: U7.GP4, U8.4B
- new net N$26: U7.GP3, U8.5B
- new net N$27: U7.GP2, U8.6B
- new net N$28: U7.GP1, U8.7B
- new net N$29: U7.GP0, U8.8B
- new net N$30: K21.S+, U8.8C
- new net N$31: K21.R+, U8.7C
- new net N$32: K11.S+, U8.6C
- new net N$33: K11.R+, U8.5C
- net 1VIN+: now also X1-2.KL; no longer X2-1.KL
- net 1VIN-: now also X1-1.KL; no longer X1-3.KL
- net 5V: now also J2.2, U10.VO; no longer MS2.5V, U6.VO
- net FONA_BAT: now also J2.4; no longer MS2.BAT
- net FONA_RST: now also J2.10; no longer MS2.RST
- net GND: now also C6.1, J2.1, K11.-, K21.-, U10.GND, U6.A0, U7.A0, U7.A1, U7.A2, U7.VSS, U8.GND; no longer MS2.GND, X1-2.KL
- net N$1: now also X1-3.KL; no longer X2-2.KL
- net N$10: now also U7.GP5, U8.3B; no longer R5.B, X4-2.KL
- net N$2: now also U7.GP7, U8.1B; no longer MS1.GPIOTX, MS2.RX
- net N$3: now also U7.GP6, U8.2B; no longer MS1.GPIORX, MS2.TX
- net N$4: now also X2-1.KL; no longer X2-3.KL
- net N$5: now also X2-3.KL; no longer X3-2.KL
- net N$6: now also X2-2.KL; no longer X3-1.KL
- net N$7: now also X3-1.KL; no longer X3-3.KL
- net N$8: now also X3-2.KL; no longer X4-1.KL
- net N$9: now also X3-3.KL; no longer X4-3.KL
- net SCL: now also R10.1, U6.SCL, U7.SCL; no longer R6.1
- net SDA: now also R11.2, U6.A1, U6.SDA, U7.SDA; no longer R7.2
- net VCC: now also C6.2, J2.3, R10.2, R11.1, U6.VS, U7.*RESET, U7.VDD; no longer MS2.VIO, R6.2, R7.1
- net VI: now also D2.C, D3.C, U10.VI, U8.COM; no longer U6.VI, X1-1.KL
Other:
- moved on the sheet: D1, J1, K1, X1-1, X1-2, X1-3, X2-1, X2-2, X2-3, X3-1, X3-2, X3-3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

Commit message: Work in progress on the main board ...
Connections:
- removed net LOUT: K22.SA, X4-3.KL
- removed net N$21: R6.A, X4-1.KL
- removed net N$9: R5.A, X3-3.KL
- new net LOUT+: K22.SA, R5.A
- new net LOUT-: R5.B, X4-3.KL
- net LIN1: now also X3-3.KL; no longer R5.B
- net LIN2: now also X4-1.KL; no longer R6.B

Commit message: Work in progress on the main board ...
Parts:
- added C7: (no value), SparkFun-Capacitors:CAP0805
- added R7: (no value), SparkFun-Resistors:RESISTOR2512
- added R8: (no value), SparkFun-Resistors:RESISTOR0805-RES
- added X6: MKDSN1,5/8-5,08, con-phoenix-508:MKDSN1,5/8-5,08
- D2, D3: value (none) -> MBRA140; device diode:SCHOTTKY-DIODESMD -> SparkFun-DiscreteSemi:DIODE-SCHOTTKY-MBRA140
- R6: value 5m -> (none); device resistor-shunt:SMV -> SparkFun-Resistors:RESISTOR0805-RES
- U7: value MCP23008-E/SS -> ATMEGA328P_TQFP; device Microchip_By_element14_Batch_1:MCP23008-E/SS -> SparkFun-DigitalIC:ATMEGA328P_TQFP
Connections:
- new net DISP1_CE: J2.8, MS1.GPIOA4
- new net DISP1_RST: J2.6, MS1.GPIOA3
- new net DISP2_CE: J2.4, MS1.GPIOA2
- new net DISP2_RST: J2.2, MS1.GPIOA1
- new net DISP_DC: J2.10, MS1.GPIOA5
- new net N$21: U7.PD7(AIN1), U8.6B
- new net N$34: J2.13
- new net N$35: J2.11
- new net N$36: J2.9
- new net N$37: D1.C, J1.1
- new net N$9: D2.C, D3.C, R7.2, U6.VIN+
- new net T_A_B: U7.PD3(INT1), X6-3.KL
- new net T_ON_OFF: U7.PD2(INT0), X6-2.KL
- net 5V: now also J2.5; no longer J2.2
- net FONA_BAT: now also J2.7; no longer J1.1, J2.4
- net FONA_RST: no longer J2.10
- net FONA_RX: now also J2.20; no longer J2.8
- net FONA_TX: now also J2.18; no longer J2.6
- net GND: now also C7.1, U7.GND@3, U7.GND@5, X4-2.KL, X6-1.KL; no longer U7.A0, U7.A1, U7.A2, U7.VSS
- net LOUT+: now also R6.2
- net MISO: now also J2.16
- net MOSI: now also J2.14
- net N$10: now also U7.PD6(AIN0), U8.7B; no longer U7.GP5, U8.3B
- net N$2: now also R6.1, R8.2, U7.PD4(XCK/T0); no longer U7.GP7, U8.1B
- net N$23: now also U7.PB0(ICP), U8.5B; no longer R6.SA, U6.VIN+
- net N$24: now also U7.PB1(OC1A), U8.4B; no longer R6.SB, U6.VIN-
- net N$25: now also U7.PB2(SS/OC1B), U8.3B; no longer U7.GP4, U8.4B
- net N$26: now also R8.1; no longer U7.GP3, U8.5B
- net N$27: now also J2.19; no longer U7.GP2, U8.6B
- net N$28: now also J2.17; no longer U7.GP1, U8.7B
- net N$29: now also J2.15; no longer U7.GP0, U8.8B
- net N$3: now also U7.PD5(T1), U8.8B; no longer U7.GP6, U8.2B
- net SCK: now also J2.12
- net SCL: now also U7.PC5(ADC5/SCL); no longer U7.SCL
- net SDA: now also U7.PC4(ADC4/SDA); no longer U7.SDA
- net VBAT: no longer D1.C
- net VCC: now also C7.2, U7.AVCC, U7.VCC@4, U7.VCC@6; no longer U7.*RESET, U7.VDD
- net VI: now also R7.1, U6.VIN-; no longer D2.C, D3.C
Other:
- moved on the sheet: D1, J1, J2, K1, K2, U8

Commit message: Update schematic
Parts:
- added K3: RT314F12, relay:RT314F12
- added R12, R13, R14, R9: (no value), SparkFun-Resistors:RESISTOR0805-RES
- added X5: MKDS_5/3-7,62, con-phoenix-mkds_5:MKDS_5/3-7,62
Connections:
- new net LIN1SENSE: K12.SA, K12.SB, R9.2
- new net LIN2SENSE: K22.OA, K22.OB, R13.2
- new net N$38: R12.2, R9.1, U7.PC1(ADC1)
- new net N$39: R12.1
- new net N$40: R13.1, R14.2, U7.PC2(ADC2)
- new net N$41: R14.1
- new net N$42: K11.S+, U8.4C
- new net N$43: K11.R+, U8.3C
- net GND: now also K31.-; no longer K11.-
- net LIN1: now also K12.PA, K12.PB, X5-1.KL; no longer K12.OB, X3-3.KL
- net LIN2: now also K22.PA, K22.PB, X5-2.KL; no longer K12.SB, X4-1.KL
- net LOUT+: now also K32.SA, K32.SB; no longer K22.SA
- net LOUT-: now also X5-3.KL; no longer X4-3.KL
- net N$2: now also U7.PC0(ADC0); no longer U7.PD4(XCK/T0)
- net N$22: now also K12.OA, K12.OB, K22.SA, K22.SB, K32.PA, K32.PB; no longer K12.PA, K22.PB
- net N$30: now also K31.S+; no longer K21.S+
- net N$31: now also K31.R+; no longer K21.R+
- net N$32: now also K21.S+; no longer K11.S+
- net N$33: now also K21.R+; no longer K11.R+
Other:
- moved on the sheet: K1, K2

Commit message: Lets hope
Parts:
- removed X4: MKDS_5/3-7,62, con-phoenix-mkds_5:MKDS_5/3-7,62
- added J3: (no value), SparkFun-Connectors:M04X2
Connections:
- net GND: now also X3-3.KL; no longer X4-2.KL
Changed lines of the file:
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@@
 <part name="X2" library="con-phoenix-mkds_5" deviceset="MKDS_5/3-" device="7,62"/>
 <part name="X3" library="con-phoenix-mkds_5" deviceset="MKDS_5/3-" device="7,62"/>
-<part name="X4" library="con-phoenix-mkds_5" deviceset="MKDS_5/3-" device="7,62"/>
 <part name="GND11" library="SparkFun-Aesthetics" deviceset="GND" device=""/>
 <part name="SUPPLY7" library="SparkFun-Aesthetics" deviceset="VCC" device=""/>
@@
 <part name="GND25" library="SparkFun-Aesthetics" deviceset="GND" device=""/>
 <part name="X5" library="con-phoenix-mkds_5" deviceset="MKDS_5/3-" device="7,62"/>
+<part name="J3" library="SparkFun-Connectors" deviceset="M04X2" device=""/>
 </parts>
 <sheets>
@@
 <instance part="X3" gate="-2" x="-137.16" y="342.9"/>
 <instance part="X3" gate="-3" x="-137.16" y="337.82"/>
-<instance part="X4" gate="-1" x="-137.16" y="330.2"/>
-<instance part="X4" gate="-2" x="-137.16" y="325.12"/>
-<instance part="X4" gate="-3" x="-137.16" y="320.04"/>
 <instance part="GND11" gate="1" x="-66.04" y="5.08" rot="R270"/>
 <instance part="SUPPLY7" gate="G$1" x="-63.5" y="10.16" rot="R90"/>
@@
 <instance part="C7" gate="G$1" x="157.48" y="335.28" rot="R90"/>
 <instance part="GND20" gate="1" x="139.7" y="335.28" rot="R270"/>
-<instance part="GND21" gate="1" x="-116.84" y="325.12" rot="R90"/>
+<instance part="GND21" gate="1" x="-116.84" y="337.82" rot="R90"/>
 <instance part="X6" gate="-1" x="208.28" y="421.64"/>
 <instance part="X6" gate="-2" x="208.28" y="416.56"/>
@@
 <instance part="X5" gate="-2" x="-137.16" y="307.34"/>
 <instance part="X5" gate="-3" x="-137.16" y="302.26"/>
+<instance part="J3" gate="G$1" x="142.24" y="302.26"/>
 </instances>
 <busses>
@@
 </segment>
 <segment>
-<pinref part="X4" gate="-2" pin="KL"/>
 <pinref part="GND21" gate="1" pin="GND"/>
-<wire x1="-132.08" y1="325.12" x2="-119.38" y2="325.12" width="0.1524" layer="91"/>
-</segment>
-<segment>
+<pinref part="X3" gate="-3" pin="KL"/>
+<wire x1="-132.08" y1="337.82" x2="-119.38" y2="337.82" width="0.1524" layer="91"/>
+</segment>
+<segment>

Commit message: Before autoroute try
Parts:
- added C8: (no value), SparkFun-Capacitors:CAP0805
- MS1: device adafruit:FEATHERWING_NODIM -> BtParts:FEATHERWING_NODIM
Connections:
- removed net N$30: K31.S+, U8.8C
- removed net N$31: K31.R+, U8.7C
- removed net N$39: R12.1
- removed net N$41: R14.1
- new net N$45: K11.S+, U8.8C
- new net N$47: K31.S+, U8.3C
- net GND: now also C8.1, K11.-, R12.1, R14.1
- net N$42: now also K31.R+; no longer K11.S+
- net N$43: now also U8.7C; no longer U8.3C
- net VCC: now also C8.2
Other:
- moved on the sheet: K1, K2, K3
Changed lines of the file:
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@@
 </classes>
 <parts>
-<part name="MS1" library="adafruit" deviceset="FEATHERWING" device="_NODIM" value="FEATHERWING_NODIM"/>
+<part name="MS1" library="BtParts" deviceset="FEATHERWING" device="_NODIM" value="FEATHERWING_NODIM"/>
 <part name="U1" library="Texas Instruments_By_element14_Batch_1" deviceset="INA219AIDR" device=""/>
 <part name="U2" library="Texas Instruments_By_element14_Batch_1" deviceset="INA219AIDR" device=""/>
@@
 <part name="X5" library="con-phoenix-mkds_5" deviceset="MKDS_5/3-" device="7,62"/>
 <part name="J3" library="SparkFun-Connectors" deviceset="M04X2" device=""/>
+<part name="C8" library="SparkFun-Capacitors" deviceset="CAP" device="0805"/>
 </parts>
 <sheets>
@@
 <instance part="R4" gate="G$1" x="-45.72" y="248.92" rot="R90"/>
 <instance part="R5" gate="G$1" x="-45.72" y="200.66" rot="R90"/>
-<instance part="K2" gate="1" x="350.52" y="330.2" rot="R90"/>
+<instance part="K2" gate="1" x="358.14" y="363.22" rot="R90"/>
 <instance part="K2" gate="2" x="226.06" y="215.9"/>
-<instance part="K3" gate="1" x="350.52" y="294.64" rot="R90"/>
+<instance part="K3" gate="1" x="358.14" y="327.66" rot="R90"/>
 <instance part="K3" gate="2" x="213.36" y="243.84"/>
 <instance part="U6" gate="A" x="22.86" y="152.4"/>
@@
 <instance part="U8" gate="A" x="292.1" y="314.96"/>
 <instance part="GND18" gate="1" x="269.24" y="292.1"/>
-<instance part="GND19" gate="1" x="363.22" y="276.86"/>
+<instance part="GND19" gate="1" x="370.84" y="309.88"/>
 <instance part="R7" gate="G$1" x="-53.34" y="152.4" rot="R90"/>
 <instance part="U7" gate="U$1" x="203.2" y="314.96"/>
@@
 <instance part="GND22" gate="1" x="271.78" y="340.36"/>
 <instance part="GND23" gate="1" x="167.64" y="421.64" rot="R270"/>
-<instance part="K1" gate="1" x="350.52" y="360.68" rot="R90"/>
+<instance part="K1" gate="1" x="358.14" y="393.7" rot="R90"/>
 <instance part="K1" gate="2" x="198.12" y="215.9"/>
 <instance part="R9" gate="G$1" x="294.64" y="373.38" rot="R90"/>
@@
 <instance part="X5" gate="-3" x="-137.16" y="302.26"/>
 <instance part="J3" gate="G$1" x="142.24" y="302.26"/>
+<instance part="C8" gate="G$1" x="157.48" y="325.12" rot="R90"/>
 </instances>
 <busses>
@@
 <segment>
 <pinref part="GND19" gate="1" pin="GND"/>
-<wire x1="363.22" y1="279.4" x2="363.22" y2="289.56" width="0.1524" layer="91"/>
+<wire x1="370.84" y1="312.42" x2="370.84" y2="322.58" width="0.1524" layer="91"/>
 <pinref part="K3" gate="1" pin="-"/>
-<wire x1="363.22" y1="289.56" x2="355.6" y2="289.56" width="0.1524" layer="91"/>
-<wire x1="363.22" y1="289.56" x2="363.22" y2="325.12" width="0.1524" layer="91"/>
-<junction x="363.22" y="289.56"/>
+<wire x1="370.84" y1="322.58" x2="363.22" y2="322.58" width="0.1524" layer="91"/>
+<wire x1="370.84" y1="322.58" x2="370.84" y2="358.14" width="0.1524" layer="91"/>
+<junction x="370.84" y="322.58"/>
 <pinref part="K2" gate="1" pin="-"/>
-<wire x1="363.22" y1="325.12" x2="355.6" y2="325.12" width="0.1524" layer="91"/>
+<wire x1="370.84" y1="358.14" x2="363.22" y2="358.14" width="0.1524" layer="91"/>
+<pinref part="K1" gate="1" pin="-"/>
+<wire x1="363.22" y1="388.62" x2="370.84" y2="388.62" width="0.1524" layer="91"/>
+<wire x1="370.84" y1="388.62" x2="370.84" y2="358.14" width="0.1524" layer="91"/>
+<junction x="370.84" y="358.14"/>
 </segment>
 <segment>
@@
 <pinref part="GND20" gate="1" pin="GND"/>
 <pinref part="C7" gate="G$1" pin="1"/>
-<wire x1="142.24" y1="335.28" x2="152.4" y2="335.28" width="0.1524" layer="91"/>
+<wire x1="142.24" y1="335.28" x2="149.86" y2="335.28" width="0.1524" layer="91"/>
+<pinref part="C8" gate="G$1" pin="1"/>
+<wire x1="149.86" y1="335.28" x2="152.4" y2="335.28" width="0.1524" layer="91"/>
+<wire x1="152.4" y1="325.12" x2="149.86" y2="325.12" width="0.1524" layer="91"/>
+<wire x1="149.86" y1="325.12" x2="149.86" y2="335.28" width="0.1524" layer="91"/>
+<junction x="149.86" y="335.28"/>
 </segment>
 <segment>
@@
 <pinref part="X6" gate="-1" pin="KL"/>
 <wire x1="170.18" y1="421.64" x2="205.74" y2="421.64" width="0.1524" layer="91"/>
+</segment>
+<segment>
+<pinref part="GND24" gate="1" pin="GND"/>
+<pinref part="R12" gate="G$1" pin="1"/>
+<wire x1="294.64" y1="342.9" x2="294.64" y2="350.52" width="0.1524" layer="91"/>
+</segment>
+<segment>
+<pinref part="GND25" gate="1" pin="GND"/>
+<pinref part="R14" gate="G$1" pin="1"/>
+<wire x1="317.5" y1="342.9" x2="317.5" y2="350.52" width="0.1524" layer="91"/>
 </segment>
 </net>
@@
 <wire x1="160.02" y1="335.28" x2="170.18" y2="335.28" width="0.1524" layer="91"/>
 <junction x="170.18" y="335.28"/>
+<pinref part="C8" gate="G$1" pin="2"/>
+<wire x1="160.02" y1="325.12" x2="170.18" y2="325.12" width="0.1524" layer="91"/>
+<wire x1="170.18" y1="325.12" x2="170.18" y2="335.28" width="0.1524" layer="91"/>
 </segment>
 </net>
@@
 <segment>
 <pinref part="U8" gate="A" pin="COM"/>
-<wire x1="309.88" y1="299.72" x2="325.12" y2="299.72" width="0.1524" layer="91"/>
+<wire x1="309.88" y1="299.72" x2="317.5" y2="299.72" width="0.1524" layer="91"/>
 <label x="314.96" y="299.72" size="1.27" layer="95"/>
 </segment>
@@
 </segment>
 </net>
-<net name="N$30" class="0">
-<segment>
-<pinref part="U8" gate="A" pin="8C"/>
-<wire x1="309.88" y1="304.8" x2="332.74" y2="304.8" width="0.1524" layer="91"/>
-<wire x1="332.74" y1="304.8" x2="332.74" y2="284.48" width="0.1524" layer="91"/>
-<pinref part="K3" gate="1" pin="S+"/>
-<wire x1="332.74" y1="284.48" x2="345.44" y2="284.48" width="0.1524" layer="91"/>
-</segment>
-</net>
-<net name="N$31" class="0">
-<segment>
-<pinref part="U8" gate="A" pin="7C"/>
-<wire x1="309.88" y1="307.34" x2="335.28" y2="307.34" width="0.1524" layer="91"/>
-<wire x1="335.28" y1="307.34" x2="335.28" y2="294.64" width="0.1524" layer="91"/>
-<pinref part="K3" gate="1" pin="R+"/>
-<wire x1="335.28" y1="294.64" x2="345.44" y2="294.64" width="0.1524" layer="91"/>
-</segment>
-</net>
 <net name="N$32" class="0">
 <segment>
 <pinref part="U8" gate="A" pin="6C"/>
-<wire x1="309.88" y1="309.88" x2="335.28" y2="309.88" width="0.1524" layer="91"/>
-<wire x1="335.28" y1="309.88" x2="335.28" y2="320.04" width="0.1524" layer="91"/>
+<wire x1="309.88" y1="309.88" x2="342.9" y2="309.88" width="0.1524" layer="91"/>
+<wire x1="342.9" y1="309.88" x2="342.9" y2="353.06" width="0.1524" layer="91"/>
 <pinref part="K2" gate="1" pin="S+"/>
-<wire x1="335.28" y1="320.04" x2="345.44" y2="320.04" width="0.1524" layer="91"/>
+<wire x1="342.9" y1="353.06" x2="353.06" y2="353.06" width="0.1524" layer="91"/>
 </segment>
 </net>
@@
 <segment>
 <pinref part="U8" gate="A" pin="5C"/>
-<wire x1="309.88" y1="312.42" x2="332.74" y2="312.42" width="0.1524" layer="91"/>
-<wire x1="332.74" y1="312.42" x2="332.74" y2="330.2" width="0.1524" layer="91"/>
+<wire x1="309.88" y1="312.42" x2="340.36" y2="312.42" width="0.1524" layer="91"/>
+<wire x1="340.36" y1="312.42" x2="340.36" y2="363.22" width="0.1524" layer="91"/>
 <pinref part="K2" gate="1" pin="R+"/>
-<wire x1="332.74" y1="330.2" x2="345.44" y2="330.2" width="0.1524" layer="91"/>
+<wire x1="340.36" y1="363.22" x2="353.06" y2="363.22" width="0.1524" layer="91"/>
 </segment>
 </net>
@@
 </segment>
 </net>
-<net name="N$39" class="0">
-<segment>
-<pinref part="R12" gate="G$1" pin="1"/>
-<wire x1="294.64" y1="350.52" x2="294.64" y2="342.9" width="0.1524" layer="91"/>
-</segment>
-</net>
 <net name="N$40" class="0">
 <segment>
@@
 </segment>
 </net>
-<net name="N$41" class="0">
-<segment>
-<pinref part="R14" gate="G$1" pin="1"/>
-<wire x1="317.5" y1="350.52" x2="317.5" y2="342.9" width="0.1524" layer="91"/>
-</segment>
-</net>
 <net name="N$42" class="0">
 <segment>
 <pinref part="U8" gate="A" pin="4C"/>
-<wire x1="309.88" y1="314.96" x2="330.2" y2="314.96" width="0.1524" layer="91"/>
-<wire x1="330.2" y1="314.96" x2="330.2" y2="350.52" width="0.1524" layer="91"/>
+<wire x1="309.88" y1="314.96" x2="337.82" y2="314.96" width="0.1524" layer="91"/>
+<wire x1="337.82" y1="314.96" x2="337.82" y2="327.66" width="0.1524" layer="91"/>
+<pinref part="K3" gate="1" pin="R+"/>
+<wire x1="337.82" y1="327.66" x2="353.06" y2="327.66" width="0.1524" layer="91"/>
+</segment>
+</net>
+<net name="N$47" class="0">
+<segment>
+<pinref part="U8" gate="A" pin="3C"/>
+<pinref part="K3" gate="1" pin="S+"/>
+<wire x1="309.88" y1="317.5" x2="353.06" y2="317.5" width="0.1524" layer="91"/>
+</segment>
+</net>
+<net name="N$43" class="0">
+<segment>
+<pinref part="K1" gate="1" pin="R+"/>
+<wire x1="345.44" y1="393.7" x2="353.06" y2="393.7" width="0.1524" layer="91"/>
+<pinref part="U8" gate="A" pin="7C"/>
+<wire x1="309.88" y1="307.34" x2="345.44" y2="307.34" width="0.1524" layer="91"/>
+<wire x1="345.44" y1="393.7" x2="345.44" y2="307.34" width="0.1524" layer="91"/>
+</segment>
+</net>
+<net name="N$45" class="0">
+<segment>
 <pinref part="K1" gate="1" pin="S+"/>
-<wire x1="330.2" y1="350.52" x2="345.44" y2="350.52" width="0.1524" layer="91"/>
-</segment>
-</net>
-<net name="N$43" class="0">
-<segment>
-<pinref part="U8" gate="A" pin="3C"/>
-<wire x1="309.88" y1="317.5" x2="325.12" y2="317.5" width="0.1524" layer="91"/>
-<wire x1="327.66" y1="317.5" x2="325.12" y2="317.5" width="0.1524" layer="91"/>
-<wire x1="325.12" y1="317.5" x2="325.12" y2="360.68" width="0.1524" layer="91"/>
-<pinref part="K1" gate="1" pin="R+"/>
-<wire x1="325.12" y1="360.68" x2="345.44" y2="360.68" width="0.1524" layer="91"/>
-</segment>
-</net>
+<wire x1="347.98" y1="383.54" x2="353.06" y2="383.54" width="0.1524" layer="91"/>
+<wire x1="347.98" y1="383.54" x2="347.98" y2="304.8" width="0.1524" layer="91"/>
+<pinref part="U8" gate="A" pin="8C"/>
+<wire x1="309.88" y1="304.8" x2="347.98" y2="304.8" width="0.1524" layer="91"/>
+</segment>
+</net>

Commit message: Schematic done. Lets route ...
Parts:
- removed J1: (no value), SparkFun-Connectors:M02PTH
- added D21, D22, D23: 3.3V, SparkFun-DiscreteSemi:DIODE-ZENER3.3V
- added R21: (no value), SparkFun-Resistors:RESISTOR0805-RES
- C7, C8: value (none) -> 0.1uF
- J2: device SparkFun-Connectors:M10X2 -> SparkFun-Connectors:M08X2
- R6: value (none) -> 10k
- renumbered R13 to R23, R9 to R22
Connections:
- net D6 renamed SD_CARD_DETECT
- removed net N$26: R8.1
- removed net N$27: J2.19
- removed net N$28: J2.17
- removed net N$29: J2.15
- removed net N$34: J2.13
- removed net N$35: J2.11
- removed net N$36: J2.9
- removed net N$37: D1.C, J1.1
- new net FONA_KEY: J2.9, MS1.GPIO12
- new net FONA_PS: J2.11, MS1.GPIOA0
- new net MASTER_EXT_IO: MS1.GPIO13, X6-8.KL
- new net N$30: U7.ADC6, U8.1B
- new net N$31: U7.ADC7, U8.2B
- new net OUT_12V_1: U8.1C, X6-4.KL
- new net OUT_12V_2: U8.2C, X6-5.KL
- new net SLAVE_EXT_IO: U7.PC3(ADC3), X6-7.KL
- new net SLAVE_GND: J3.6
- new net SLAVE_MISO: J3.1, U7.PB4(MISO)
- new net SLAVE_MOSI: J3.4, U7.PB3(MOSI/OC2)
- new net SLAVE_NOTIFY: MS1.GPIO5, U7.PD4(XCK/T0)
- new net SLAVE_RESET: J3.5, MS1.GPIO11, R6.1, U7.PC6(/RESET)
- new net SLAVE_RX: J3.7, U7.PD0(RXD)
- new net SLAVE_SCK: J3.3, U7.PB5(SCK)
- new net SLAVE_TX: J3.8, U7.PD1(TXD)
- new net SLAVE_VCC: J3.2
- net FONA_RX: now also J2.15; no longer J2.20
- net FONA_TX: now also J2.13; no longer J2.18
- net GND: now also D21.A, D22.A, D23.A, R8.1, U7.AGND
- net LOUT+: now also R21.2; no longer R6.2
- net LOUT-: now also X6-6.KL
- net N$2: now also D21.C, R21.1; no longer R6.1
- net N$38: now also D22.C
- net N$40: now also D23.C
- net VBAT: now also D1.C; no longer J1.2
- net VCC: now also R6.2
Other:
- moved on the sheet: J3, R12, R14, R6, R8
