File: Hardware/SolarMonitorMainBoard/SolarMonitorMainBoard.sch (EAGLE design)
At the start: 50 parts, among them K1 RT314F12, K2 RT314F12, K3 RT314F12, U1 INA219AIDR, U10 TSR_1-2450, U2 INA219AIDR, U3 INA219AIDR, U4 INA219AIDR, U5 INA219AIDR, U6 INA219AIDR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

Commit message: Some Routing
Parts:
- removed R14, R8: (no value), SparkFun-Resistors:RESISTOR0805-RES
- added R13, R42: (no value), SparkFun-Resistors:RESISTOR0805-RES
- renumbered R10 to R41
Connections:
- net FONA_RX: now also J2.13; no longer J2.15
- net FONA_TX: now also J2.15; no longer J2.13
- net GND: now also R21.1, R22.1, R23.1; no longer R12.1, R14.1, R8.1
- net LIN1SENSE: now also R12.2; no longer R22.2
- net LIN2SENSE: now also R13.2; no longer R23.2
- net LOUT+: now also R11.2; no longer R21.2
- net N$2: now also R11.1, R21.2; no longer R21.1, R8.2
- net N$38: now also R12.1, R22.2; no longer R12.2, R22.1
- net N$40: now also R13.1, R23.2; no longer R14.2, R23.1
- net SDA: now also R42.2; no longer R11.2
- net VCC: now also R42.1; no longer R11.1
Other:
- moved on the sheet: R11, R12, R21, R22, R23
Changed lines of the file:
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@@
 <part name="SUPPLY4" library="SparkFun-Aesthetics" deviceset="VCC" device=""/>
 <part name="SUPPLY5" library="SparkFun-Aesthetics" deviceset="VCC" device=""/>
-<part name="R10" library="SparkFun-Resistors" deviceset="RESISTOR" device="0805-RES"/>
-<part name="R11" library="SparkFun-Resistors" deviceset="RESISTOR" device="0805-RES"/>
+<part name="R41" library="SparkFun-Resistors" deviceset="RESISTOR" device="0805-RES"/>
+<part name="R42" library="SparkFun-Resistors" deviceset="RESISTOR" device="0805-RES"/>
 <part name="SUPPLY6" library="SparkFun-Aesthetics" deviceset="VCC" device=""/>
 <part name="C1" library="SparkFun-Capacitors" deviceset="CAP" device="0805"/>
@@
 <part name="GND21" library="SparkFun-Aesthetics" deviceset="GND" device=""/>
 <part name="X6" library="con-phoenix-508" deviceset="MKDSN1,5/8-5,08" device=""/>
+<part name="R11" library="SparkFun-Resistors" deviceset="RESISTOR" device="0805-RES"/>
 <part name="R21" library="SparkFun-Resistors" deviceset="RESISTOR" device="0805-RES"/>
-<part name="R8" library="SparkFun-Resistors" deviceset="RESISTOR" device="0805-RES"/>
 <part name="GND22" library="SparkFun-Aesthetics" deviceset="GND" device=""/>
 <part name="GND23" library="SparkFun-Aesthetics" deviceset="GND" device=""/>
 <part name="K1" library="relay" deviceset="RT?F*" device="314" technology="12"/>
+<part name="R12" library="SparkFun-Resistors" deviceset="RESISTOR" device="0805-RES"/>
 <part name="R22" library="SparkFun-Resistors" deviceset="RESISTOR" device="0805-RES"/>
-<part name="R12" library="SparkFun-Resistors" deviceset="RESISTOR" device="0805-RES"/>
 <part name="GND24" library="SparkFun-Aesthetics" deviceset="GND" device=""/>
+<part name="R13" library="SparkFun-Resistors" deviceset="RESISTOR" device="0805-RES"/>
 <part name="R23" library="SparkFun-Resistors" deviceset="RESISTOR" device="0805-RES"/>
-<part name="R14" library="SparkFun-Resistors" deviceset="RESISTOR" device="0805-RES"/>
 <part name="GND25" library="SparkFun-Aesthetics" deviceset="GND" device=""/>
 <part name="X5" library="con-phoenix-mkds_5" deviceset="MKDS_5/3-" device="7,62"/>
@@
 <instance part="SUPPLY4" gate="G$1" x="0" y="261.62"/>
 <instance part="SUPPLY5" gate="G$1" x="0" y="213.36"/>
-<instance part="R10" gate="G$1" x="7.62" y="58.42"/>
-<instance part="R11" gate="G$1" x="38.1" y="58.42"/>
+<instance part="R41" gate="G$1" x="7.62" y="58.42"/>
+<instance part="R42" gate="G$1" x="38.1" y="58.42"/>
 <instance part="SUPPLY6" gate="G$1" x="22.86" y="63.5"/>
 <instance part="C1" gate="G$1" x="-10.16" y="401.32" rot="R90"/>
@@
 <instance part="X6" gate="-7" x="208.28" y="391.16"/>
 <instance part="X6" gate="-8" x="208.28" y="386.08"/>
-<instance part="R21" gate="G$1" x="271.78" y="373.38" rot="R90"/>
-<instance part="R8" gate="G$1" x="271.78" y="350.52" rot="R90"/>
+<instance part="R11" gate="G$1" x="271.78" y="373.38" rot="R90"/>
+<instance part="R21" gate="G$1" x="271.78" y="350.52" rot="R90"/>
 <instance part="GND22" gate="1" x="271.78" y="340.36"/>
 <instance part="GND23" gate="1" x="167.64" y="421.64" rot="R270"/>
 <instance part="K1" gate="1" x="358.14" y="393.7" rot="R90"/>
 <instance part="K1" gate="2" x="198.12" y="215.9"/>
-<instance part="R22" gate="G$1" x="294.64" y="373.38" rot="R90"/>
-<instance part="R12" gate="G$1" x="294.64" y="350.52" rot="R90"/>
+<instance part="R12" gate="G$1" x="294.64" y="373.38" rot="R90"/>
+<instance part="R22" gate="G$1" x="294.64" y="350.52" rot="R90"/>
 <instance part="GND24" gate="1" x="294.64" y="340.36"/>
-<instance part="R23" gate="G$1" x="317.5" y="373.38" rot="R90"/>
-<instance part="R14" gate="G$1" x="317.5" y="350.52" rot="R90"/>
+<instance part="R13" gate="G$1" x="317.5" y="373.38" rot="R90"/>
+<instance part="R23" gate="G$1" x="317.5" y="350.52" rot="R90"/>
 <instance part="GND25" gate="1" x="317.5" y="340.36"/>
 <instance part="X5" gate="-1" x="-137.16" y="312.42"/>
@@
 <segment>
 <pinref part="GND24" gate="1" pin="GND"/>
-<pinref part="R12" gate="G$1" pin="1"/>
+<pinref part="R22" gate="G$1" pin="1"/>
 <wire x1="294.64" y1="342.9" x2="294.64" y2="345.44" width="0.1524" layer="91"/>
 <pinref part="D22" gate="G$1" pin="A"/>
@@
 <segment>
 <pinref part="GND25" gate="1" pin="GND"/>
-<pinref part="R14" gate="G$1" pin="1"/>
+<pinref part="R23" gate="G$1" pin="1"/>
 <wire x1="317.5" y1="342.9" x2="317.5" y2="345.44" width="0.1524" layer="91"/>
 <pinref part="D23" gate="G$1" pin="A"/>
@@
 </segment>
 <segment>
-<pinref part="R8" gate="G$1" pin="1"/>
+<pinref part="R21" gate="G$1" pin="1"/>
 <pinref part="GND22" gate="1" pin="GND"/>
 <wire x1="271.78" y1="345.44" x2="271.78" y2="342.9" width="0.1524" layer="91"/>
@@
 </segment>
 <segment>
-<pinref part="R10" gate="G$1" pin="2"/>
+<pinref part="R41" gate="G$1" pin="2"/>
 <pinref part="SUPPLY6" gate="G$1" pin="VCC"/>
 <wire x1="12.7" y1="58.42" x2="22.86" y2="58.42" width="0.1524" layer="91"/>
 <wire x1="22.86" y1="58.42" x2="22.86" y2="63.5" width="0.1524" layer="91"/>
-<pinref part="R11" gate="G$1" pin="1"/>
+<pinref part="R42" gate="G$1" pin="1"/>
 <wire x1="33.02" y1="58.42" x2="22.86" y2="58.42" width="0.1524" layer="91"/>
 </segment>
@@
 <wire x1="-2.54" y1="195.58" x2="-2.54" y2="152.4" width="0.1524" layer="91"/>
 <label x="-2.54" y="53.34" size="1.778" layer="95" rot="R180" xref="yes"/>
-<pinref part="R10" gate="G$1" pin="1"/>
+<pinref part="R41" gate="G$1" pin="1"/>
 <wire x1="-2.54" y1="152.4" x2="-2.54" y2="58.42" width="0.1524" layer="91"/>
 <wire x1="-2.54" y1="58.42" x2="-2.54" y2="53.34" width="0.1524" layer="91"/>
@@
 <wire x1="48.26" y1="208.28" x2="48.26" y2="160.02" width="0.1524" layer="91"/>
 <label x="48.26" y="53.34" size="1.778" layer="95" rot="R180" xref="yes"/>
-<pinref part="R11" gate="G$1" pin="2"/>
+<pinref part="R42" gate="G$1" pin="2"/>
 <wire x1="48.26" y1="160.02" x2="48.26" y2="121.92" width="0.1524" layer="91"/>
 <wire x1="48.26" y1="120.396" x2="48.26" y2="58.42" width="0.1524" layer="91"/>
@@
 </segment>
 <segment>
-<pinref part="J2" gate="G$1" pin="15"/>
-<wire x1="-119.38" y1="-17.78" x2="-129.54" y2="-17.78" width="0.1524" layer="91"/>
-<label x="-129.54" y="-17.78" size="1.27" layer="95"/>
+<pinref part="J2" gate="G$1" pin="13"/>
+<wire x1="-129.54" y1="-15.24" x2="-119.38" y2="-15.24" width="0.1524" layer="91"/>
+<label x="-129.54" y="-15.24" size="1.27" layer="95"/>
 </segment>
 </net>
@@
 </segment>
 <segment>
-<pinref part="R21" gate="G$1" pin="2"/>
+<pinref part="R11" gate="G$1" pin="2"/>
 <wire x1="271.78" y1="378.46" x2="271.78" y2="383.54" width="0.1524" layer="91"/>
 <wire x1="271.78" y1="383.54" x2="279.4" y2="383.54" width="0.1524" layer="91"/>
@@
 <net name="N$2" class="0">
 <segment>
-<pinref part="R21" gate="G$1" pin="1"/>
-<pinref part="R8" gate="G$1" pin="2"/>
+<pinref part="R11" gate="G$1" pin="1"/>
+<pinref part="R21" gate="G$1" pin="2"/>
 <wire x1="271.78" y1="368.3" x2="271.78" y2="365.76" width="0.1524" layer="91"/>
 <wire x1="271.78" y1="365.76" x2="271.78" y2="355.6" width="0.1524" layer="91"/>
@@
 </segment>
 <segment>
-<pinref part="R22" gate="G$1" pin="2"/>
+<pinref part="R12" gate="G$1" pin="2"/>
 <wire x1="294.64" y1="378.46" x2="294.64" y2="383.54" width="0.1524" layer="91"/>
 <wire x1="294.64" y1="383.54" x2="307.34" y2="383.54" width="0.1524" layer="91"/>
@@
 </segment>
 <segment>
-<pinref part="R23" gate="G$1" pin="2"/>
+<pinref part="R13" gate="G$1" pin="2"/>
 <wire x1="317.5" y1="378.46" x2="317.5" y2="383.54" width="0.1524" layer="91"/>
 <wire x1="317.5" y1="383.54" x2="327.66" y2="383.54" width="0.1524" layer="91"/>
@@
 <net name="N$38" class="0">
 <segment>
-<pinref part="R22" gate="G$1" pin="1"/>
-<pinref part="R12" gate="G$1" pin="2"/>
+<pinref part="R12" gate="G$1" pin="1"/>
+<pinref part="R22" gate="G$1" pin="2"/>
 <wire x1="294.64" y1="368.3" x2="294.64" y2="365.76" width="0.1524" layer="91"/>
 <wire x1="294.64" y1="365.76" x2="294.64" y2="355.6" width="0.1524" layer="91"/>
@@
 <net name="N$40" class="0">
 <segment>
-<pinref part="R23" gate="G$1" pin="1"/>
-<pinref part="R14" gate="G$1" pin="2"/>
+<pinref part="R13" gate="G$1" pin="1"/>
+<pinref part="R23" gate="G$1" pin="2"/>
 <wire x1="317.5" y1="368.3" x2="317.5" y2="365.76" width="0.1524" layer="91"/>
 <wire x1="317.5" y1="365.76" x2="317.5" y2="355.6" width="0.1524" layer="91"/>
@@
 </segment>
 <segment>
-<pinref part="J2" gate="G$1" pin="13"/>
-<wire x1="-119.38" y1="-15.24" x2="-129.54" y2="-15.24" width="0.1524" layer="91"/>
-<label x="-129.54" y="-15.24" size="1.27" layer="95"/>
-</segment>
-</net>
+<pinref part="J2" gate="G$1" pin="15"/>
+<wire x1="-119.38" y1="-17.78" x2="-129.54" y2="-17.78" width="0.1524" layer="91"/>
+<label x="-129.54" y="-17.78" size="1.27" layer="95"/>
+</segment>
+</net>

Commit message: More routing
Connections:
- removed net SLAVE_GND: J3.6
- removed net SLAVE_VCC: J3.2
- net GND: now also J3.6
- net N$30: now also U7.ADC7; no longer U7.ADC6
- net N$31: now also U7.ADC6; no longer U7.ADC7
- net VCC: now also J3.2
Changed lines of the file:
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@@
 <junction x="271.78" y="342.9"/>
+</segment>
+<segment>
+<pinref part="J3" gate="G$1" pin="6"/>
+<wire x1="121.92" y1="297.18" x2="142.24" y2="297.18" width="0.1524" layer="91"/>
+<label x="124.46" y="297.18" size="1.27" layer="95"/>
 </segment>
 </net>
@@
 <pinref part="R6" gate="G$1" pin="2"/>
 <wire x1="147.32" y1="363.22" x2="147.32" y2="360.68" width="0.1524" layer="91"/>
+</segment>
+<segment>
+<pinref part="J3" gate="G$1" pin="2"/>
+<wire x1="121.92" y1="302.26" x2="142.24" y2="302.26" width="0.1524" layer="91"/>
+<label x="124.46" y="302.26" size="1.27" layer="95"/>
 </segment>
 </net>
@@
 </segment>
 </net>
-<net name="SLAVE_VCC" class="0">
-<segment>
-<pinref part="J3" gate="G$1" pin="2"/>
-<wire x1="121.92" y1="302.26" x2="142.24" y2="302.26" width="0.1524" layer="91"/>
-<label x="124.46" y="302.26" size="1.27" layer="95"/>
-</segment>
-</net>
 <net name="SLAVE_MOSI" class="0">
 <segment>
@@
 </segment>
 </net>
-<net name="SLAVE_GND" class="0">
-<segment>
-<pinref part="J3" gate="G$1" pin="6"/>
-<wire x1="121.92" y1="297.18" x2="142.24" y2="297.18" width="0.1524" layer="91"/>
-<label x="124.46" y="297.18" size="1.27" layer="95"/>
-</segment>
-</net>
 <net name="SLAVE_TX" class="0">
 <segment>
@@
 <net name="N$30" class="0">
 <segment>
-<pinref part="U7" gate="U$1" pin="ADC6"/>
-<wire x1="226.06" y1="330.2" x2="266.7" y2="330.2" width="0.1524" layer="91"/>
-<wire x1="266.7" y1="330.2" x2="266.7" y2="322.58" width="0.1524" layer="91"/>
 <pinref part="U8" gate="A" pin="1B"/>
+<wire x1="266.7" y1="327.66" x2="266.7" y2="322.58" width="0.1524" layer="91"/>
 <wire x1="266.7" y1="322.58" x2="274.32" y2="322.58" width="0.1524" layer="91"/>
+<pinref part="U7" gate="U$1" pin="ADC7"/>
+<wire x1="226.06" y1="327.66" x2="266.7" y2="327.66" width="0.1524" layer="91"/>
 </segment>
 </net>
 <net name="N$31" class="0">
 <segment>
-<pinref part="U7" gate="U$1" pin="ADC7"/>
-<wire x1="226.06" y1="327.66" x2="264.16" y2="327.66" width="0.1524" layer="91"/>
-<wire x1="264.16" y1="327.66" x2="264.16" y2="320.04" width="0.1524" layer="91"/>
+<wire x1="264.16" y1="330.2" x2="264.16" y2="320.04" width="0.1524" layer="91"/>
 <pinref part="U8" gate="A" pin="2B"/>
 <wire x1="264.16" y1="320.04" x2="274.32" y2="320.04" width="0.1524" layer="91"/>
-</segment>
-</net>
+<pinref part="U7" gate="U$1" pin="ADC6"/>
+<wire x1="264.16" y1="330.2" x2="226.06" y2="330.2" width="0.1524" layer="91"/>
+</segment>
+</net>

Commit message: Fix Warnings ADD I2C to header
Parts:
- J2: device SparkFun-Connectors:M08X2 -> SparkFun-Connectors:M10X2
Connections:
- net FONA_RST: now also J2.17
- net SCL: now also J2.18
- net SDA: now also J2.20
Changed lines of the file:
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@@
 <part name="D2" library="SparkFun-DiscreteSemi" deviceset="DIODE-SCHOTTKY" device="-MBRA140" value="MBRA140"/>
 <part name="D3" library="SparkFun-DiscreteSemi" deviceset="DIODE-SCHOTTKY" device="-MBRA140" value="MBRA140"/>
-<part name="J2" library="SparkFun-Connectors" deviceset="M08X2" device=""/>
+<part name="J2" library="SparkFun-Connectors" deviceset="M10X2" device=""/>
 <part name="GND12" library="SparkFun-Aesthetics" deviceset="GND" device=""/>
 <part name="SUPPLY11" library="SparkFun-Aesthetics" deviceset="VCC" device=""/>
@@
 <pinref part="U1" gate="A" pin="A0"/>
 <wire x1="2.54" y1="388.62" x2="5.08" y2="388.62" width="0.1524" layer="91"/>
+<junction x="2.54" y="386.08"/>
+<junction x="2.54" y="378.46"/>
 </segment>
 <segment>
@@
 <wire x1="5.08" y1="340.36" x2="2.54" y2="340.36" width="0.1524" layer="91"/>
 <wire x1="2.54" y1="340.36" x2="2.54" y2="330.2" width="0.1524" layer="91"/>
+<junction x="2.54" y="330.2"/>
 </segment>
 <segment>
@@
 <pinref part="U3" gate="A" pin="A1"/>
 <wire x1="2.54" y1="292.1" x2="5.08" y2="292.1" width="0.1524" layer="91"/>
+<junction x="2.54" y="284.48"/>
 </segment>
 <segment>
@@
 <pinref part="U5" gate="A" pin="A0"/>
 <wire x1="2.54" y1="198.12" x2="5.08" y2="198.12" width="0.1524" layer="91"/>
+<junction x="2.54" y="187.96"/>
 </segment>
 <segment>
@@
 <pinref part="U$1" gate="G$1" pin="VSS"/>
 <wire x1="-45.72" y1="-78.74" x2="-33.02" y2="-78.74" width="0.1524" layer="91"/>
+<junction x="-45.72" y="-86.36"/>
+<junction x="-45.72" y="-83.82"/>
 </segment>
 <segment>
@@
 <pinref part="U6" gate="A" pin="A0"/>
 <wire x1="2.54" y1="149.86" x2="5.08" y2="149.86" width="0.1524" layer="91"/>
+<junction x="2.54" y="139.7"/>
 </segment>
 <segment>
@@
 <pinref part="C1" gate="G$1" pin="2"/>
 <wire x1="0" y1="401.32" x2="-7.62" y2="401.32" width="0.1524" layer="91"/>
+<junction x="0" y="401.32"/>
 </segment>
 <segment>
@@
 <pinref part="C2" gate="G$1" pin="2"/>
 <wire x1="0" y1="353.06" x2="-7.62" y2="353.06" width="0.1524" layer="91"/>
+<junction x="0" y="350.52"/>
+<junction x="0" y="353.06"/>
 </segment>
 <segment>
@@
 <pinref part="C3" gate="G$1" pin="2"/>
 <wire x1="-7.62" y1="307.34" x2="0" y2="307.34" width="0.1524" layer="91"/>
+<junction x="0" y="304.8"/>
+<junction x="0" y="307.34"/>
 </segment>
 <segment>
@@
 <pinref part="C4" gate="G$1" pin="2"/>
 <wire x1="-7.62" y1="259.08" x2="0" y2="259.08" width="0.1524" layer="91"/>
+<junction x="0" y="246.38"/>
+<junction x="0" y="256.54"/>
+<junction x="0" y="259.08"/>
 </segment>
 <segment>
@@
 <pinref part="C5" gate="G$1" pin="2"/>
 <wire x1="-7.62" y1="210.82" x2="0" y2="210.82" width="0.1524" layer="91"/>
+<junction x="0" y="210.82"/>
 </segment>
 <segment>
@@
 <pinref part="R42" gate="G$1" pin="1"/>
 <wire x1="33.02" y1="58.42" x2="22.86" y2="58.42" width="0.1524" layer="91"/>
+<junction x="22.86" y="58.42"/>
 </segment>
 <segment>
@@
 <pinref part="C6" gate="G$1" pin="2"/>
 <wire x1="-7.62" y1="162.56" x2="0" y2="162.56" width="0.1524" layer="91"/>
+<junction x="0" y="162.56"/>
 </segment>
 <segment>
@@
 <pinref part="U6" gate="A" pin="SCL"/>
 <wire x1="5.08" y1="152.4" x2="-2.54" y2="152.4" width="0.1524" layer="91"/>
+<wire x1="-2.54" y1="147.32" x2="-2.54" y2="152.4" width="0.1524" layer="91"/>
+<junction x="-2.54" y="152.4"/>
+<junction x="-2.54" y="58.42"/>
+<junction x="-2.54" y="195.58"/>
+<junction x="-2.54" y="200.66"/>
+<junction x="-2.54" y="297.18"/>
+<junction x="-2.54" y="342.9"/>
+<junction x="-2.54" y="248.92"/>
 </segment>
 <segment>
@@
 <wire x1="226.06" y1="332.74" x2="241.3" y2="332.74" width="0.1524" layer="91"/>
 <label x="228.6" y="332.74" size="1.27" layer="95"/>
+</segment>
+<segment>
+<pinref part="J2" gate="G$1" pin="18"/>
+<wire x1="-104.14" y1="-20.32" x2="-90.17" y2="-20.32" width="0.1524" layer="91"/>
+<label x="-102.362" y="-20.066" size="1.27" layer="95"/>
 </segment>
 </net>
@@
 <label x="48.26" y="53.34" size="1.778" layer="95" rot="R180" xref="yes"/>
 <pinref part="R42" gate="G$1" pin="2"/>
-<wire x1="48.26" y1="160.02" x2="48.26" y2="121.92" width="0.1524" layer="91"/>
-<wire x1="48.26" y1="120.396" x2="48.26" y2="58.42" width="0.1524" layer="91"/>
+<wire x1="48.26" y1="160.02" x2="48.26" y2="122.936" width="0.1524" layer="91"/>
+<wire x1="48.26" y1="122.936" x2="48.26" y2="58.42" width="0.1524" layer="91"/>
 <wire x1="48.26" y1="58.42" x2="48.26" y2="53.34" width="0.1524" layer="91"/>
 <wire x1="43.18" y1="58.42" x2="48.26" y2="58.42" width="0.1524" layer="91"/>
@@
 <pinref part="U6" gate="A" pin="A1"/>
 <wire x1="5.08" y1="147.32" x2="-1.016" y2="147.32" width="0.1524" layer="91"/>
-<wire x1="-1.016" y1="147.32" x2="-1.016" y2="120.396" width="0.1524" layer="91"/>
-<wire x1="-1.016" y1="120.396" x2="48.26" y2="120.396" width="0.1524" layer="91"/>
-<wire x1="48.26" y1="120.396" x2="48.26" y2="121.92" width="0.1524" layer="91"/>
+<wire x1="-1.016" y1="147.32" x2="-1.016" y2="122.936" width="0.1524" layer="91"/>
+<wire x1="-1.016" y1="122.936" x2="48.26" y2="122.936" width="0.1524" layer="91"/>
+<junction x="48.26" y="58.42"/>
+<junction x="48.26" y="350.52"/>
+<junction x="48.26" y="304.8"/>
+<junction x="48.26" y="256.54"/>
+<junction x="48.26" y="208.28"/>
+<junction x="48.26" y="160.02"/>
+<junction x="48.26" y="122.936"/>
 </segment>
 <segment>
@@
 <wire x1="226.06" y1="335.28" x2="241.3" y2="335.28" width="0.1524" layer="91"/>
 <label x="228.6" y="335.28" size="1.27" layer="95"/>
+</segment>
+<segment>
+<pinref part="J2" gate="G$1" pin="20"/>
+<wire x1="-104.14" y1="-22.86" x2="-89.916" y2="-22.86" width="0.1524" layer="91"/>
+<label x="-102.362" y="-22.86" size="1.27" layer="95"/>
 </segment>
 </net>
@@
 <pinref part="J2" gate="G$1" pin="5"/>
 <wire x1="-139.7" y1="-5.08" x2="-119.38" y2="-5.08" width="0.1524" layer="91"/>
+<junction x="-15.24" y="48.26"/>
 </segment>
 </net>
@@
 <label x="7.62" y="-15.24" size="1.27" layer="95"/>
 </segment>
+<segment>
+<pinref part="J2" gate="G$1" pin="17"/>
+<wire x1="-119.38" y1="-20.32" x2="-129.54" y2="-20.32" width="0.1524" layer="91"/>
+<label x="-129.54" y="-20.32" size="1.27" layer="95"/>
+</segment>
 </net>
 <net name="VBAT" class="0">
@@
 <pinref part="R5" gate="G$1" pin="SB"/>
 <wire x1="-43.18" y1="190.5" x2="-43.18" y2="193.04" width="0.1524" layer="91"/>
-</segment>
-</net>
-<net name="SCL1" class="0">
-<segment>
-<wire x1="-2.54" y1="147.32" x2="-2.54" y2="152.4" width="0.1524" layer="91"/>
 </segment>
 </net>
@@
 </sheet>
 </sheets>
+<errors>
+</errors>
 </schematic>
 </drawing>
